File: kicad/tos-io.kicad_sch (KiCad schematic)
At the start: 25 parts, among them J1 RaspPi Pin Header, J2 DE9_Receptacle, J3 Keyboard, J4 Mouse, J5 Conn_02x06_Odd_Even, SW1 STATUS, U1 MAX232

Commit message: Add breakout header on TOS I/O board
Parts:
- removed J5: Conn_02x06_Odd_Even, Connector_PinSocket_2.54mm:PinSocket_2x06_P2.54mm_Vertical, symbol Connector_Generic:Conn_02x06_Odd_Even
- added J5: PMOD SPI 2A, Library:PinSocket_2x06_Top_Bottom_P2.54mm_Vertical, symbol Connector_Generic:Conn_02x06_Top_Bottom
- added J6: Conn_01x07, Connector_PinHeader_2.54mm:PinHeader_1x07_P2.54mm_Vertical, symbol Connector_Generic:Conn_01x07
Connections:
- net +3V3: now also J5.12 (Pin_12), J5.6 (Pin_6)
- net GND: now also J5.11 (Pin_11), J5.5 (Pin_5), J6.1 (Pin_1)
- net GPIO_7: no longer J4.1, R8.1
- net RX: now also J6.6 (Pin_6)
- net TX: now also J6.7 (Pin_7)
- net PMOD_2_MOSI: now reaches J1.19 (Pin_19)
- net PMOD_2_MOSI: now also J5.2 (Pin_2)
- net PMOD_3_MISO: now reaches J1.21 (Pin_21)
- net PMOD_3_MISO: now also J5.3 (Pin_3)
- net PMOD_4_SCK: now reaches J1.23 (Pin_23)
- net PMOD_4_SCK: now also J5.4 (Pin_4)
- net PS2_MOUSE_DATA: now reaches J1.27 (Pin_27)
- net PS2_MOUSE_DATA: now also J4.1, R8.1
- net PS2_MOUSE_CLK: now reaches J1.28 (Pin_28)
- net PS2_MOUSE_CLK: now also J4.5, R7.1
- net GPIO_12 renamed PMOD_7_INT
- net PMOD_7_INT: now also J5.7 (Pin_7)
- net GPIO_13: no longer names the net of J1.33 (Pin_33)
- net GPIO_14 renamed TXTTL
- net GPIO_15 renamed RXTTL
- net GPIO_16 renamed PMOD_8_RESET
- net PMOD_8_RESET: now also J5.8 (Pin_8)
- net GPIO_17 renamed LED_BLUE
- net LED_BLUE: now also R3.1; no longer R2.1
- net GPIO_19: no longer names the net of J1.35 (Pin_35)
- net GPIO_2 renamed BUTTON
- net BUTTON: now also J1.15 (Pin_15), J6.2 (Pin_2); no longer J1.3 (Pin_3)
- net GPIO_20 renamed PMOD_9
- net PMOD_9: now also J5.9 (Pin_9)
- net GPIO_21 renamed PMOD_10
- net PMOD_10: now also J5.10 (Pin_10)
- net GPIO_22 renamed LED_RED
- net LED_RED: now also J1.3 (Pin_3), J6.3 (Pin_3); no longer J1.15 (Pin_15)
- net GPIO_23 renamed PS2_CLK
- net PS2_CLK: now also J6.5 (Pin_5)
- net GPIO_24 renamed PS2_DATA
- net PS2_DATA: now also J6.4 (Pin_4)
- net GPIO_26: no longer names the net of J1.37 (Pin_37)
- net GPIO_27 renamed LED_GREEN
- net LED_GREEN: now also R2.1; no longer R3.1
- net GPIO_6: no longer names the net of J1.31 (Pin_31)
- removed net GPIO_8: J1.24 (Pin_24), J4.5, R7.1
- new net PMOD_1_SS: J1.24 (Pin_24), J5.1 (Pin_1)
- no-connect marks 21 -> 20
